File: nTerm2-s.kicad_sch (KiCad schematic)
At the start: 107 parts, among them J1 VGA, J2 Keyboard, J3 Mouse, J4 Speaker, J5 DE9_Plug_MountingHoles, J6 USB_C_Receptacle_USB2.0_16P, K1 IM41 3V, K2 IM41 3V, K3 IM41 3V, Q1 BC817, Q2 BC817, Q3 BC817, Q4 BC817, Q5 BC817, SW1 IO0, SW2 RESET, SW3 DEFAULTS, U1 ESP32-WROOM-32, U2 LM386, U3 MAX3232E, U4 CP2102N-Axx-xQFN28, U5 NCP1117-3.3_SOT223

Commit message: v0.04
Parts:
- C23: value 100u -> 100u/25V
- U4: footprint Package_DFN_QFN:QFN-28-1EP_5x5mm_P0.5mm_EP3.35x3.35mm -> Package_DFN_QFN:QFN-28-1EP_5x5mm_P0.5mm_EP3.35x3.35mm_handsolder
Other:
- note added: "For original CP2102 (not CP2102N), don't place R40, and use 0OHM for R39"
Changed lines of the file:
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@@
 	(title_block
 		(title "nTerm2-s")
-		(date "2025-01-30")
-		(rev "0.03")
+		(date "2025-02-19")
+		(rev "0.04")
 		(company "Sporos Tech ₍^•_•^₎ﾉ")
 		(comment 1 "Peter de Vroomen")
@@
 		)
 	)
+	(rectangle
+		(start 71.12 85.09)
+		(end 91.44 109.22)
+		(stroke
+			(width 0.1016)
+			(type dash)
+			(color 255 0 0 1)
+		)
+		(fill
+			(type color)
+			(color 255 0 0 0.1254901961)
+		)
+	)
+	(text "For original CP2102\n(not CP2102N), don't\nplace R40, and use\n0OHM for R39"
+		(exclude_from_sim no)
+		(at 80.772 78.486 0)
+		(effects
+			(font
+				(size 1.27 1.27)
+				(color 255 0 0 1)
+			)
+		)
+	)
 	(label "_RTS_DTR"
 		(at 179.07 252.73 0)
@@
 			)
 		)
-		(property "Footprint" "Package_DFN_QFN:QFN-28-1EP_5x5mm_P0.5mm_EP3.35x3.35mm"
+		(property "Footprint" "Package_DFN_QFN:QFN-28-1EP_5x5mm_P0.5mm_EP3.35x3.35mm_handsolder"
 			(at 140.97 154.94 0)
 			(effects
@@
 			)
 		)
-		(property "Value" "100u"
+		(property "Value" "100u/25V"
 			(at 224.282 164.338 0)
 			(effects
@@
 		)
 		(property "Value" "5K"
-			(at 246.7259 117.0939 0)
+			(at 257.81 27.432 0)
 			(effects
 				(font

Commit message: nTerm2-S v0.05 - New PCBs ordered.
Parts:
- removed D5, D7, D9: BAT43W-V, Diode_SMD:D_SOD-123, symbol Diode:BAT43W-V
- added Q6, Q7, Q8: BC817, Package_TO_SOT_SMD:SOT-23, symbol Transistor_BJT:BC817
- added R41, R42, R43: 1K, Resistor_SMD:R_0603_1608Metric_Pad0.98x0.95mm_HandSolder, symbol Device:R
- D1, D2: footprint Diode_SMD:D_SMA -> Diode_SMD:D_SMA_Handsoldering; symbol Diode:P4SMAJ5.0CA -> Sporos_Tech:P4SMAJ5.0CA
- D11, D12: footprint LED_THT:DIALIGHT_LED_3MM_DOUBLE -> Sporos_Tech_Footprints:DIALIGHT_LED_3MM_DOUBLE
- D4: footprint LED_THT:DIALIGHT_LED_3MM_SINGLE -> Sporos_Tech_Footprints:DIALIGHT_LED_3MM_SINGLE; symbol Device:LED pins reversed -> Sporos_Tech:LED pins reversed
- J1: footprint Connector_Dsub:DSUB-15-HD_Female_Horizontal_P2.29x1.98mm_EdgePinOffset8.35mm_Housed_MountingHolesOffset10.89mm -> Sporos_Tech_Footprints:DSUB-15-HD_Female_Horizontal_P2.29x1.98mm_EdgePinOffset3.03mm_Housed_MountingHolesOffset4.94mm
- J2, J3: symbol Connector:Mini-DIN-6 -> Sporos_Tech:Mini-DIN-6-alt
- J4: footprint Connector_Audio:Jack_3.5mm_Ledino_KB3SPRS_Horizontal -> Sporos_Tech_Footprints:Jack_3.5mm_Ledino_KB3SPRS_Horizontal-alt
- J5: footprint Connector_Dsub:DSUB-9_Male_Horizontal_P2.77x2.84mm_EdgePinOffset4.94mm_Housed_MountingHolesOffset7.48mm -> Sporos_Tech_Footprints:DSUB-9_Male_Horizontal_P2.77x2.84mm_EdgePinOffset4.94mm_Housed_MountingHolesOffset7.48mm
- J6: footprint Connector_USB:USB_C_Receptacle_Molex_213716-0001 -> Sporos_Tech_Footprints:USB_C_Receptacle_Molex_213716-0001
- K1, K2, K3: footprint Relay_SMD:Relay_DPDT_AXICOM_IMSeries_Gullwing -> Sporos_Tech_Footprints:Relay_DPDT_AXICOM_IMSeries_Gullwing
- R32, R33, R34: value 3K9 -> 2K2
- SW1, SW2, SW3: footprint Button_Switch_THT:SW_Tactile_SPST_Angled_PTS645Vx58-2LFS -> Sporos_Tech_Footprints:SW_Tactile_SPST_Angled_PTS645Vx58-2LFS-alt
- U4: footprint Package_DFN_QFN:QFN-28-1EP_5x5mm_P0.5mm_EP3.35x3.35mm_handsolder -> Sporos_Tech_Footprints:QFN-28-1EP_5x5mm_P0.5mm_EP3.35x3.35mm_handsolder
Connections:
- net +5V: now also Q6.3 (C), Q7.3 (C), Q8.3 (C)
- net GND: now also J4.S; no longer J4.G (1)
- net REVERSE_RTS_CTS_DTR_DSR: now also R42.1
- net REVERSE_RX_TX: now also R41.1
- net RTS_CTS_OR_DTR_DSR: now also R43.1
- net at C26.1, Q4.3 (C), R33.1: now also Q7.2 (E)
- net at C27.1, Q5.3 (C), R34.1: now also Q8.2 (E)
- net at C25.1, Q3.3 (C), R32.1: now also Q6.2 (E)
- new net: Q6.1 (B), R41.2
- new net: Q7.1 (B), R42.2
- new net: Q8.1 (B), R43.2
Other:
- moved on the sheet: C26, C27, D10, D8, R33, R34
