File: nTerm2-s.kicad_sch (KiCad schematic)
At the start: 110 parts, among them J1 VGA, J2 Keyboard, J3 Mouse, J4 Speaker, J5 DE9_Plug_MountingHoles, J6 USB_C_Receptacle_USB2.0_16P, K1 IM41 3V, K2 IM41 3V, K3 IM41 3V, Q1 BC817, Q2 BC817, Q3 BC817, Q4 BC817, Q5 BC817, Q6 BC817, Q7 BC817, Q8 BC817, SW1 IO0, SW2 RESET, SW3 DEFAULTS, U1 ESP32-WROOM-32, U2 LM386, U3 MAX3232E, U4 CP2102N-Axx-xQFN28, U5 NCP1117-3.3_SOT223

Commit message: V0.06 - Use USBLC6-2 for ESD protection, instead of those big TVS diodes. Those big TVS diodes were a bad choice, they have far too high a capacity for USB 2.0 use. Removed resistors from the bases of Q6, Q7 and Q8 as it only works reliably with very low resistance, and we might as well make them 0 ohm then. Added bypass capability for the audio amplifier, giving the user a choice to assemble it and drive a speaker, or save some money, don't assemble it and use line-out. Also a choice to solder a jackplug for external audio or use a connector for internal speaker.
Parts:
- removed D1, D2: P4SMAJ5.0CA, Diode_SMD:D_SMA_Handsoldering, symbol Sporos_Tech:P4SMAJ5.0CA
- removed R41, R42, R43: 1K, Resistor_SMD:R_0603_1608Metric_Pad0.98x0.95mm_HandSolder, symbol Device:R
- added J7: Line-out/Speaker, Connector_PinHeader_2.54mm:PinHeader_1x02_P2.54mm_Vertical, symbol Connector_Generic:Conn_01x02
- added JP1: Bypass, Jumper:SolderJumper-3_P1.3mm_Open_RoundedPad1.0x1.5mm_NumberLabels, symbol Jumper:SolderJumper_3_Open
- added U6: USBLC6-2SC6, Package_TO_SOT_SMD:SOT-23-6, symbol Power_Protection:USBLC6-2SC6
- J4: value Speaker -> Line-out/Speaker
- J5: value DE9_Plug_MountingHoles -> RS-232 V.24
Connections:
- net +5V: now also U6.5 (VBUS)
- net GND: now also J7.2 (Pin_2), U6.2 (GND)
- net REVERSE_RTS_CTS_DTR_DSR: now also Q7.1 (B)
- net REVERSE_RX_TX: now also Q6.1 (B)
- net RTS_CTS_OR_DTR_DSR: now also Q8.1 (B)
- net at J6.A6 (D+), J6.B6 (D+): now also U6.4 (I/O2); no longer U4.4 (D+)
- net at C1.2, J4.T: now also J7.1 (Pin_1), JP1.3 (B)
- net at R19.2, U2.2 (-): now also JP1.1 (A); no longer C3.2
- net at J6.A7 (D-), J6.B7 (D-): now also U6.6 (I/O1); no longer U4.5 (D-)
- new net: U4.5 (D-), U6.1 (I/O1)
- new net: U4.4 (D+), U6.3 (I/O2)
- new net: C3.2, JP1.2 (C)
Other:
- note added: "* For CP2102 original, bridge R39 (make 0 Ohm) and don't place R40. * For CP2102N, place resistors as drawn."
- note added: "Bypass: You can choose to use line-out or provide an audio amplifier. * Solder bridge 1-2 and assemble all components inside the red box to implement the audio amplifier and drive a speaker directly. * Solder bridge 2-3, and leave out all components inside the red box to have only a line-out. Then assemble J4 or J7 as needed. Or don't assemble any and just solder wires directly to the PCB."
- note added: "You can choose to assemble either J4 or J7, depending on if you want to bring the audio 'outside' or keep it internal."
- note removed: "For original CP2102 (not CP2102N), don't place R40, and use 0OHM for R39"
- moved on the sheet: C1, C13, C14, C15, C16, C17, C18, C19, C2, C20, C21, C22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

Commit message: Update capacitor footprint to larger size.
Parts:
- C23: footprint Capacitor_Tantalum_SMD:CP_EIA-6032-28_Kemet-C_Pad2.25x2.35mm_HandSolder -> Capacitor_Tantalum_SMD:CP_EIA-7343-30_AVX-N_Pad2.25x2.55mm_HandSolder
Changed lines of the file:
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@@
 			)
 		)
-		(property "Footprint" "Capacitor_Tantalum_SMD:CP_EIA-6032-28_Kemet-C_Pad2.25x2.35mm_HandSolder"
+		(property "Footprint" "Capacitor_Tantalum_SMD:CP_EIA-7343-30_AVX-N_Pad2.25x2.55mm_HandSolder"
 			(at 98.7552 36.83 0)
 			(effects

Commit message: Some small updates, a fix, and exported all libraries into the project, for distribution.
Parts:
- C1, C10, C11, C12, C13, C14, C17, C18, C19, C2, C20, C21, C23, C25, C26, C27, C8, C9: symbol Device:C_Polarized -> Library:C_Polarized
- C15, C16, C22, C24, C3, C4, C5, C6, C7: symbol Device:C -> Library:C
- D10, D6, D8: symbol Diode:BAT43W-V -> Library:BAT43W-V
- D11, D12: symbol Device:LED_Dual_AKAK -> Library:LED_Dual_AKAK
- D3: symbol Diode:1N5819 -> Library:1N5819
- D4: symbol Sporos_Tech:LED pins reversed -> Library:LED pins reversed
- H1, H2, H3, H4, H5, H6: symbol Mechanical:MountingHole -> Library:MountingHole
- J1: symbol Connector:DE15_Receptacle_HighDensity_MountingHoles -> Library:DE15_Receptacle_HighDensity_MountingHoles
- J2, J3: symbol Sporos_Tech:Mini-DIN-6-alt -> Library:Mini-DIN-6-alt
- J4: symbol Connector_Audio:AudioJack2_Ground_Switch -> Library:AudioJack2_Ground_Switch
- J5: symbol Connector:DE9_Plug_MountingHoles -> Library:DE9_Plug_MountingHoles
- J6: symbol Connector:USB_C_Receptacle_USB2.0_16P -> Library:USB_C_Receptacle_USB2.0_16P
- J7: symbol Connector_Generic:Conn_01x02 -> Library:Conn_01x02
- JP1: symbol Jumper:SolderJumper_3_Open -> Library:SolderJumper_3_Open
- K1, K2, K3: symbol Relay:IM41 -> Library:IM41
- Q1, Q2, Q3, Q4, Q5, Q6, Q7, Q8: symbol Transistor_BJT:BC817 -> Library:BC817
- R1, R10, R11, R12, R13, R14, R15, R16, R17, R18, R19, R2, R20, R21, R22, R23, R24, R25, R26, R27, R28, R29, R3, R30, R31, R32, R33, R34, R35, R36, R37, R38, R39, R4, R40, R5, R6, R7, R8, R9: symbol Device:R -> Library:R
- SW1, SW2, SW3: symbol Switch:CK_KMS2xxGP -> Library:CK_KMS2xxGP
- U1: symbol RF_Module:ESP32-WROOM-32 -> Library:ESP32-WROOM-32
- U2: symbol Amplifier_Audio:LM386 -> Library:LM386
- U3: symbol Custom_Symbols_Library:MAX3232E -> Library:MAX3232E
- U4: symbol Interface_USB:CP2102N-Axx-xQFN28 -> Library:CP2102N-Axx-xQFN28
- U5: symbol Regulator_Linear:NCP1117-3.3_SOT223 -> Library:NCP1117-3.3_SOT223
- U6: symbol Power_Protection:USBLC6-2SC6 -> Library:USBLC6-2SC6
